File: circuit_boards/main_VCO_board/kicad_7/power_supply.kicad_sch (KiCad schematic)
At the start: 63 parts, among them J4 power_entry, U1 TL072, U10 TL072, U1002 L78L05_SOT89, U1003 L79L05_SOT89, U1005 LM4040DBZ-5, U11 TL072, U12 LM324, U13 NE5532, U14 TL072, U15 TL072, U3 TL072, U5 TL072, U6 SSI2130, U7 TL072, U8 SSI2130, U9 4013

Commit message: Progress on circuit boards
Parts:
- R1002: value ? -> 4k7
Changed lines of the file:
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@@
   (title_block
     (title "MICRO-OX Main VCO board")
-    (date "2023-03-27")
+    (date "2023-04-12")
     (rev "0")
     (comment 2 "creativecommons.org/licenses/by/4.0")
@@
   (symbol (lib_id "Device:R") (at 187.96 127 0) (unit 1)
     (in_bom yes) (on_board yes) (dnp no) (fields_autoplaced)
-    (property "Reference" "R1002" (at 190.5 125.73 0)
+    (property "Reference" "R1002" (at 190.5 126.365 0)
       (effects (font (size 1.27 1.27)) (justify left))
     )
-    (property "Value" "?" (at 190.5 128.27 0)
+    (property "Value" "4k7" (at 190.5 128.905 0)
       (effects (font (size 1.27 1.27)) (justify left))
     )
