File: circuit_boards/modulation_board/kicad_7/power_supply.kicad_sch (KiCad schematic)
At the start: 27 parts, among them J6 power_entry, U201 SSI2130, U202 TL072, U301 TL072, U501 L78L05_SOT89, U502 L79L05_SOT89, U503 LM4040C-2.5

Commit message: Progress on circuit boards
Parts:
- removed C507, C508, C509, C510, C511, C512, C513: 100n, Capacitor_SMD:C_0805_2012Metric, symbol Device:C
- removed R501: 1k8, Resistor_SMD:R_0805_2012Metric, symbol Device:R
- removed TP506: 2v5_ref, TestPoint:TestPoint_Keystone_5000-5004_Miniature, symbol Connector:TestPoint
- removed U202, U301: TL072, Package_SO:SO-8_5.3x6.2mm_P1.27mm, symbol Amplifier_Operational:TL072
- removed U503: LM4040C-2.5, Package_TO_SOT_SMD:SOT-23, symbol Reference_Voltage:LM4040DBZ-2.5
- added C1007: 2u2, Capacitor_SMD:C_0805_2012Metric, symbol Device:C
- added C1008, C1009, C1010, C1011, C1012, C1013, C1014, C1015, C1016, C1017, C1018: 100n, Capacitor_SMD:C_0603_1608Metric, symbol Device:C
- added FB1001, FB1002: 100R @ 100MHz, Inductor_SMD:L_0805_2012Metric, symbol Device:FerriteBead_Small
- added TP1006: 3v3, TestPoint:TestPoint_Keystone_5000-5004_Miniature, symbol Connector:TestPoint
- added U10, U13, U14: TL072, Package_SO:SOIC-8_3.9x4.9mm_P1.27mm, symbol Amplifier_Operational:TL072
- added U1003: L78L33_SOT89, Package_TO_SOT_SMD:SOT-89-3, symbol Regulator_Linear:L78L33_SOT89
- added U15 (x2): MCP6002-xSN, Package_SO:SOIC-8_3.9x4.9mm_P1.27mm, symbol Amplifier_Operational:MCP6002-xSN
- C1005: renamed from C503; footprint Capacitor_SMD:C_0805_2012Metric -> Capacitor_SMD:C_0603_1608Metric
- C1006: renamed from C504; footprint Capacitor_SMD:C_0805_2012Metric -> Capacitor_SMD:C_0603_1608Metric
- J4: renamed from J6; footprint Connector_IDC:IDC-Header_2x05_P2.54mm_Vertical -> custom_footprints:10_pin_IDC-Header
- renumbered C505 to C1001, C506 to C1002, C501 to C1003, C502 to C1004, TP501 to TP1001, TP502 to TP1002, TP503 to TP1003, TP504 to TP1004, TP505 to TP1005, U501 to U1001, U502 to U1002, U201 to U12
Connections:
- net +5V: now also C1017.1, FB1001.1
- net -5V: now also C1018.2
- net GND: now also C1007.2, C1008.2, C1009.2, C1010.1, C1011.2, C1012.1, C1013.2, C1014.1, C1015.2, C1016.2, C1017.2, C1018.1, U1003.2 (GND)
- net +15V renamed +12V
- net +12V: now also C1009.1, C1011.1, C1013.1, U10.8 (V+), U13.8 (V+), U14.8 (V+)
- net -15V renamed -12V
- net -12V: now also C1010.2, C1012.2, C1014.2, U10.4 (V-), U13.4 (V-), U14.4 (V-)
- new net: C1007.1, FB1001.2, U1003.3 (IN)
- new net +3.3V: C1008.1, C1015.1, C1016.1, FB1002.1, TP1006.1, U1003.1 (OUT)
- new net +3.3VA: FB1002.2
Other:
- note removed: "2130 Decoupling"
- note removed: "2130 Power"
- note removed: "Bulk Decoupling"
- note removed: "Opamp Decoupling"
- note removed: "Opamp Power"
- moved on the sheet: C1001, C1002, C1003, C1004, C1005, C1006, J4, TP1001, TP1002, TP1003, TP1004, TP1005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
