File: circuit_boards/modulation_board/kicad_7/DAC.kicad_sch (KiCad schematic)
At the start: 58 parts, among them U10 TL072, U503 LM4040C-2.5, U8 DAC8162xDGSx, U803 MCP6002-xSN, U9 DAC128S085CIMT

Commit message: Add potentiometer 3d model to VCO and MOD boards
Parts:
- RV?: footprint Potentiometer_THT:Potentiometer_Alpha_RD901F-40-00D_Single_Vertical -> custom_footprints:Potentiometer_Alpha_RD901F-40-00D_Single_Vertical
Changed lines of the file:
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@@
       (effects (font (size 1.27 1.27)) (justify right))
     )
-    (property "Footprint" "Potentiometer_THT:Potentiometer_Alpha_RD901F-40-00D_Single_Vertical" (at 213.36 133.35 0)
+    (property "Footprint" "custom_footprints:Potentiometer_Alpha_RD901F-40-00D_Single_Vertical" (at 213.36 133.35 0)
       (effects (font (size 1.27 1.27)) hide)
     )
