File: circuit_boards/modulation_board/kicad_7/analog_controls.kicad_sch (KiCad schematic)
At the start: 29 parts, among them U5 74HC4067PW

Commit message: Add potentiometer 3d model to VCO and MOD boards
Parts:
- RV401, RV402, RV403, RV404, RV405, RV406, RV407, RV408, RV412: footprint Potentiometer_THT:Potentiometer_Alpha_RD901F-40-00D_Single_Vertical -> custom_footprints:Potentiometer_Alpha_RD901F-40-00D_Single_Vertical
Changed lines of the file:
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@@
     (comment 4 "Author: Jordan Aceto")
   )
+  (bus_alias "SPI" (members "SCK" "SDO" "~{CS_0}" "~{CS_1}" "~{CS_2}"))
   (bus_alias "MUX" (members "S0" "S1" "S2" "S3" "COM_ANALOG" "COM_DISCRETE"))
   (bus_alias "" (members ))
-  (bus_alias "SPI" (members "SCK" "SDO" "~{CS_0}" "~{CS_1}" "~{CS_2}"))
   (junction (at 139.7 44.45) (diameter 0) (color 0 0 0 0)
   )
@@
       (effects (font (size 1.27 1.27)) (justify right))
     )
-    (property "Footprint" "Potentiometer_THT:Potentiometer_Alpha_RD901F-40-00D_Single_Vertical" (at 38.1 45.72 0)
+    (property "Footprint" "custom_footprints:Potentiometer_Alpha_RD901F-40-00D_Single_Vertical" (at 38.1 45.72 0)
       (effects (font (size 1.27 1.27)) hide)
     )
@@
       (effects (font (size 1.27 1.27)) (justify right))
     )
-    (property "Footprint" "Potentiometer_THT:Potentiometer_Alpha_RD901F-40-00D_Single_Vertical" (at 38.1 68.58 0)
+    (property "Footprint" "custom_footprints:Potentiometer_Alpha_RD901F-40-00D_Single_Vertical" (at 38.1 68.58 0)
       (effects (font (size 1.27 1.27)) hide)
     )
@@
       (effects (font (size 1.27 1.27)) (justify right))
     )
-    (property "Footprint" "Potentiometer_THT:Potentiometer_Alpha_RD901F-40-00D_Single_Vertical" (at 38.1 91.44 0)
+    (property "Footprint" "custom_footprints:Potentiometer_Alpha_RD901F-40-00D_Single_Vertical" (at 38.1 91.44 0)
       (effects (font (size 1.27 1.27)) hide)
     )
@@
       (effects (font (size 1.27 1.27)) (justify right))
     )
-    (property "Footprint" "Potentiometer_THT:Potentiometer_Alpha_RD901F-40-00D_Single_Vertical" (at 83.82 91.44 0)
+    (property "Footprint" "custom_footprints:Potentiometer_Alpha_RD901F-40-00D_Single_Vertical" (at 83.82 91.44 0)
       (effects (font (size 1.27 1.27)) hide)
     )
@@
       (effects (font (size 1.27 1.27)) (justify right))
     )
-    (property "Footprint" "Potentiometer_THT:Potentiometer_Alpha_RD901F-40-00D_Single_Vertical" (at 83.82 45.72 0)
+    (property "Footprint" "custom_footprints:Potentiometer_Alpha_RD901F-40-00D_Single_Vertical" (at 83.82 45.72 0)
       (effects (font (size 1.27 1.27)) hide)
     )
@@
       (effects (font (size 1.27 1.27)) (justify right))
     )
-    (property "Footprint" "Potentiometer_THT:Potentiometer_Alpha_RD901F-40-00D_Single_Vertical" (at 83.82 68.58 0)
+    (property "Footprint" "custom_footprints:Potentiometer_Alpha_RD901F-40-00D_Single_Vertical" (at 83.82 68.58 0)
       (effects (font (size 1.27 1.27)) hide)
     )
@@
       (effects (font (size 1.27 1.27)) (justify right))
     )
-    (property "Footprint" "Potentiometer_THT:Potentiometer_Alpha_RD901F-40-00D_Single_Vertical" (at 38.1 114.3 0)
+    (property "Footprint" "custom_footprints:Potentiometer_Alpha_RD901F-40-00D_Single_Vertical" (at 38.1 114.3 0)
       (effects (font (size 1.27 1.27)) hide)
     )
@@
       (effects (font (size 1.27 1.27)) (justify right))
     )
-    (property "Footprint" "Potentiometer_THT:Potentiometer_Alpha_RD901F-40-00D_Single_Vertical" (at 129.54 119.38 0)
+    (property "Footprint" "custom_footprints:Potentiometer_Alpha_RD901F-40-00D_Single_Vertical" (at 129.54 119.38 0)
       (effects (font (size 1.27 1.27)) hide)
     )
@@
       (effects (font (size 1.27 1.27)) (justify right))
     )
-    (property "Footprint" "Potentiometer_THT:Potentiometer_Alpha_RD901F-40-00D_Single_Vertical" (at 83.82 114.3 0)
-      (effects (font (size 1.27 1.27)) hide)
-    )
+    (property "Footprint" "custom_footprints:Potentiometer_Alpha_RD901F-40-00D_Single_Vertical" (at 83.82 114.3 0)
+      (effects (font (size 1.27 1.27)) hide)
+    )
