File: front_panel/kicad_7/micro_ox_front_panel.kicad_sch (KiCad schematic)
At the start: 1 part

Commit message: Progress on circuit boards
Parts:
- removed TP1: dummy, TestPoint:TestPoint_Keystone_5000-5004_Miniature, symbol Connector:TestPoint
- added H1, H2, H3, H4, H5, H6, H7, H8: MountingHole_Pad, MountingHole:MountingHole_3.2mm_M3_Pad_Via, symbol Mechanical:MountingHole_Pad
Connections:
- net GND: now also H1.1, H2.1, H3.1, H4.1, H5.1, H6.1, H7.1, H8.1

Commit message: Update front panel
Other:
- moved on the sheet: H1, H2, H3, H4, H5, H6, H7, H8
