File: circuit_boards/VCF_VCA_board/kicad_7/power_supply.kicad_sch (KiCad schematic)
At the start: 37 parts, among them J4 power_entry, U1 TL072, U2 TL072, U3 TL072, U4 TL072, U5 TL072, U6 TL072, U7 TL072, U707 LM4040DBZ-5, U8 SSI2140, U9 SSI2164

Commit message: Progress on circuit boards
Parts:
- R701: value ? -> 2k7
Changed lines of the file:
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@@
   (title_block
     (title "MICRO-OX VCF/VCA board")
-    (date "2023-03-21")
+    (date "2023-04-13")
     (rev "0")
     (comment 1 "creativecommons.org/licenses/by/4.0/")
@@
       (effects (font (size 1.27 1.27)) (justify left))
     )
-    (property "Value" "?" (at 176.53 110.49 0)
-      (effects (font (size 1.27 1.27)) (justify left))
-    )
+    (property "Value" "2k7" (at 176.53 110.49 0)
+      (effects (font (size 1.27 1.27)) (justify left))
+    )
