File: circuit_boards/VCF_VCA_board/kicad_7/VCF_VCA_board.kicad_pcb (KiCad board)
At the start: 2 copper layers, 60.3 x 165.1 mm, 138 parts, among them J1 VCO_BOARD_CON, J2 MOD_BOARD_CON, J3 VCF_EXT_CON, J4 power_entry, SW1 SR1712F-0204, SW2 E-Switch_EG2201B, SW3 E-Switch_EG2301, SW4 E-Switch_EG2201B, U1 TL072, U2 TL072, U3 TL072, U4 TL072, U5 TL072, U6 TL072, U7 TL072, U707 LM4040DBZ-5, U8 SSI2140, U9 SSI2164

Commit message: Tone down Q-compensation to avoid volume increase with high Q
Parts:
- R217: value 18k -> 30k
Changed lines of the file:
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@@
         (effects (font (size 1 1) (thickness 0.15)) (justify mirror))
     )
-    (fp_text value "18k" (at 0 -1.43) (layer "B.Fab")
+    (fp_text value "30k" (at 0 -1.43) (layer "B.Fab")
         (effects (font (size 1 1) (thickness 0.15)) (justify mirror))
     )
